Commit message: imu publishing, caster wheels

File: resource/robot_model.urdf (robot description, URDF)
Before this commit: robot /home/daniel/ros2_ws/src/third_webots_pkg/resource/robot_model.urdf, 6 links, 5 joints
Links:
- added link front caster wheel; collision sphere radius=0.015; visual sphere radius=0.015
- added link imu
- added link rear caster wheel; collision sphere radius=0.015; visual sphere radius=0.015
Joints:
- added joint base_link_imu_joint: type fixed, parent base_link, child imu, origin xyz=0 0 0.082 rpy=0 0 0
- added joint hingejoint: type continuous, parent base_link, child rear caster wheel, origin xyz=0.03 0 0.005 rpy=0 0.003543 0, axis 0 1 0
- added joint hingejoint_0: type continuous, parent base_link, child front caster wheel, origin xyz=-0.03 0 0.005 rpy=0 0 0, axis 0 1 0
- joint left wheel motor: origin xyz=0 -0.045 0.025 rpy=0 1.49585 0 -> xyz=0 -0.045 0.015 rpy=0 0 0
- joint right wheel motor: origin xyz=0 0 0.025 rpy=0 -0.862703 0 -> xyz=0 0 0.015 rpy=0 0 0
